Commit message: rviz包改名为urdf包。修正里程计bug

File: pi_catkin_ws/src/tinypibot_urdf/urdf/my_car_camera.urdf (robot description, URDF)
Before this commit: robot my_car_camera, 9 links, 8 joints
Links:
- link base_footprint: geometry visual sphere radius=0.1
Joints:
- joint base_link2base_footprint: child base_link -> base_footprint; parent base_footprint -> base_link

Commit message: 上下位机增加uart通讯模式

File: pi_catkin_ws/src/tinypibot_urdf/urdf/my_car_camera.urdf (robot description, URDF)
Before this commit: robot my_car_camera, 9 links, 8 joints
Joints:
- joint base_link2base_footprint: child base_footprint -> base_link; parent base_link -> base_footprint
